File: Eagle/Tarjeta.sch (EAGLE design)
At the start: 49 parts, among them IC1 DSPIC30F4011-30I_P, IC2 LM321LVIDCKR, IC3 LMT86QDCKRQ1, IC4 TXB0108PWR, Q1 TIP41C, T1 2N2222, T10 2N2222, T2 2N2222, T3 2N2222, T4 2N2222, T5 2N2222, T6 2N2222, T7 2N2222, T8 2N2222, T9 2N2222

Commit message: Esquematico
se actulizo el esquematico
Parts:
- added IC5: LORA_MOTE, LORA_MOTE:LORA_MOTE
- added J2, J3: TBL002A-350-03GR-2OR, TBL002A-350-03GR-2OR:TBL002A-350-03GR-2OR
- IC2: value LM321LVIDCKR -> LM324LVIDR; device LM321LVIDCKR:LM321LVIDCKR -> LM324LVIDR:LM324LVIDR
- J1: value (none) -> TBL002A-350-03GR-2OR; device con-amp:MTA02-100 -> TBL002A-350-03GR-2OR:TBL002A-350-03GR-2OR
- R1, R3, R4, R5: value (none) -> RC0805FR-071KL; device rcl:R-EU_0207/10 -> RC0805FR-071KL:RC0805FR-071KL
- R10, R11, R12, R13, R14, R6, R7, R8, R9: value ERA6AEB101V -> RC0805FR-071KL; device ERA6AEB101V:ERA6AEB101V -> RC0805FR-071KL:RC0805FR-071KL
- R15, R16: value ERA6AEB101V -> (none); device ERA6AEB101V:ERA6AEB101V -> rcl:R-EU_0204/7
- R2: value (none) -> ERA-6VEB1002V; device rcl:R-EU_0207/10 -> ERA-6VEB1002V:ERA-6VEB1002V
- T1, T10, T2, T3, T4, T5, T6, T7, T8, T9: value 2N2222 -> 2N3904; device transistor:2N2222 -> transistor-neu-to92:2N3904
Connections:
- removed net N$1: D1.A, J1.2, Q1.C
- removed net N$6 (its old number): IC2.IN-, R15.1, R16.2
- new net FAN1: D1.C, J2.A2
- new net FAN2: D1.A, J2.B1, Q1.C
- new net GND1: T10.E, T9.E
- new net RESISTENCIA: IC2.IN1-, R15.2, R16.2
- net AVAILABLE: now also R3.2; no longer R5.2
- net GATE_UP: now also R5.2; no longer R3.2
- net GND: now also IC5.GND, J1.A1, R15.1; no longer R15.2, T10.E, T9.E
- net LMT86: now also IC2.IN1+; no longer IC2.IN+
- net POT_LINEAR: now also J3.A1
- net RX_LORA: now also IC5.UARTTX
- net SONAR_ADC: now also J2.A1
- net SONAR_SERIAL: now also J1.A2
- net TEMP: now also IC2.OUT1; no longer IC2.OUT
- net TX_LORA: now also IC5.UARTRX
- net V5: now also IC5.V5, J1.B1; no longer D1.C, J1.1

Commit message: 16/05/2021
actualizacion
Parts:
- added C2, C3, C4: C0805X104K1RAC3316, C0805X104K1RAC3316:C0805X104K1RAC3316
- added J4: 172447-0004, 172447-0004:172447-0004
- added LED10: 599-0181-007F, 599-0181-007F:599-0181-007F
- added R18: RC0805FR-071KL, RC0805FR-071KL:RC0805FR-071KL
- added T11: 2N3904, transistor-neu-to92:2N3904
Connections:
- new net GND2: T11.E
- new net LED10: IC1.!FLTA!/INT0/RE8, T11.B
- new net N$1: LED10.K, T11.C
- new net N$22: LED10.A, R18.1
- new net V1: R18.2
- net AVAILABLE: now also IC1.OC3/RD2; no longer IC1.OC4/RD3
- net GATE_DOWN: now also IC1.OC4/RD3; no longer IC1.EMUD2/OC2/IC2/INT2/RD1
- net GATE_UP: now also IC1.EMUD2/OC2/IC2/INT2/RD1; no longer IC1.!FLTA!/INT0/RE8
- net GND: now also C2.1, C3.1, C4.1, J4.3
- net LED7: now also IC1.OSC2/CLKO/RC15
- net LED8: now also IC1.EMUD1/SOSCI/T2CK/U1ATX/CN1/RC13
- net LED9: now also IC1.EMUC1/SOSCO/T1CK/U1ARX/CN0/RC14
- net V5: now also C2.2, C3.2, C4.2, J4.4
Other:
- moved on the sheet: J1, J2, J3, LED9, R14, R15, R16, T10
